File: elec/layout/base/smart-knob.kicad_pcb (KiCad board)
At the start: 2 copper layers, 81.2 x 81.2 mm, 73 parts

Commit message: base layout 40% complete
Parts:
- added Z5: dummy_keepouts, view_custom:ViewKeepouts3d, F.Cu at (61.4, 61.0)
- C20, C21, C22, C23, C24, C25, C26, C27, C28, C29: value 16V 100nF X7R ±10% 0402 Multilayer Ceramic Capacitors MLCC - SMD/SMT ROHS -> 25V 1uF X5R ±10% 0402 Multilayer Ceramic Capacitors MLCC - SMD/SMT ROHS
- U15: renamed from L1; value 3.3uH ±10% 1206 Inductors (SMD) ROHS -> 3.3 +/- 0.99 (30%) microhenry; footprint lib:L1206 -> lib:IND-SMD_L1.2-W0.7
- U17: renamed from U16; footprint lib:LED-SMD_4P-L2.0-W2.0-BR -> lib:LED-SMD_4P-L4.0-W1.4_SK6805SIDE-S
- U18: renamed from U17; footprint lib:LED-SMD_4P-L2.0-W2.0-BR -> lib:LED-SMD_4P-L4.0-W1.4_SK6805SIDE-S
- U19: renamed from U18; footprint lib:LED-SMD_4P-L2.0-W2.0-BR -> lib:LED-SMD_4P-L4.0-W1.4_SK6805SIDE-S
- U20: renamed from U19; footprint lib:LED-SMD_4P-L2.0-W2.0-BR -> lib:LED-SMD_4P-L4.0-W1.4_SK6805SIDE-S
- U21: renamed from U20; footprint lib:LED-SMD_4P-L2.0-W2.0-BR -> lib:LED-SMD_4P-L4.0-W1.4_SK6805SIDE-S
- U22: renamed from U21; footprint lib:LED-SMD_4P-L2.0-W2.0-BR -> lib:LED-SMD_4P-L4.0-W1.4_SK6805SIDE-S
- U23: renamed from U22; footprint lib:LED-SMD_4P-L2.0-W2.0-BR -> lib:LED-SMD_4P-L4.0-W1.4_SK6805SIDE-S
- U24: renamed from U23; footprint lib:LED-SMD_4P-L2.0-W2.0-BR -> lib:LED-SMD_4P-L4.0-W1.4_SK6805SIDE-S
- U25: renamed from U24; footprint lib:LED-SMD_4P-L2.0-W2.0-BR -> lib:LED-SMD_4P-L4.0-W1.4_SK6805SIDE-S
- U26: renamed from U25; footprint lib:LED-SMD_4P-L2.0-W2.0-BR -> lib:LED-SMD_4P-L4.0-W1.4_SK6805SIDE-S
- moved C7 187.0 mm to (62.7, 64.8), turned to 180 degrees
- moved U6 165.7 mm to (61.4, 61.0), turned to 90 degrees
- moved U16 157.1 mm to (40.0, 52.3), turned to 90 degrees
- moved C19 156.6 mm to (42.8, 52.4), turned to 90 degrees
- moved R11 155.7 mm to (37.8, 61.0), turned to 180 degrees
- moved R9 143.2 mm to (45.6, 61.0), turned to 180 degrees
- moved C3 138.3 mm to (26.6, 80.5)
- moved U4 138.3 mm to (23.8, 85.4)
- moved C4 138.3 mm to (25.1, 80.4)
- moved C5 138.3 mm to (23.0, 80.4)
- moved R3 138.3 mm to (26.0, 83.2)
- moved U3 138.3 mm to (37.0, 88.8)
- moved R7 125.2 mm to (78.2, 95.7)
- moved R10 107.1 mm to (77.2, 61.0), turned to 180 degrees
- moved C20 103.7 mm to (116.7, 37.4), turned to 0 degrees
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- renumbered U15 to U16
Connections:
- net led1.ic-vcc-1 renamed led1-vcc
- R11 pad 1: usbc-gnd -> n
- R11 pad 2: p2 -> usbc-gnd
- R14 pad 1: usbc-gnd -> n
- R9 pad 2: usbc-gnd -> n
- U17 pad 2: led1.ic-vcc -> usbc-gnd
- U17 pad 3: usbc-gnd -> led1-vcc-1
- U18 pad 2: led2.ic-vcc -> usbc-gnd
- U18 pad 3: usbc-gnd -> led2-vcc
- U18 pad 4: led1.ic-vcc -> led1-vcc-1
- U19 pad 2: led3.ic-vcc -> usbc-gnd
- U19 pad 3: usbc-gnd -> led3-vcc
- U19 pad 4: led2.ic-vcc -> led2-vcc
- U20 pad 2: led4.ic-vcc -> usbc-gnd
- U20 pad 3: usbc-gnd -> led4-vcc
- U20 pad 4: led3.ic-vcc -> led3-vcc
- U21 pad 2: led5.ic-vcc -> usbc-gnd
- U21 pad 3: usbc-gnd -> led5-vcc
- U21 pad 4: led4.ic-vcc -> led4-vcc
- U22 pad 2: led6.ic-vcc -> usbc-gnd
- U22 pad 3: usbc-gnd -> led6-vcc
- U22 pad 4: led5.ic-vcc -> led5-vcc
- U23 pad 2: led7.ic-vcc -> usbc-gnd
- U23 pad 3: usbc-gnd -> led7-vcc
- U23 pad 4: led6.ic-vcc -> led6-vcc
- U24 pad 2: led8.ic-vcc -> usbc-gnd
- U24 pad 3: usbc-gnd -> led8-vcc
- U24 pad 4: led7.ic-vcc -> led7-vcc
- U25 pad 2: led9.ic-vcc -> usbc-gnd
- U25 pad 3: usbc-gnd -> led9-vcc
- U25 pad 4: led8.ic-vcc -> led8-vcc
- U26 pad 2: led10.ic-vcc -> usbc-gnd
- U26 pad 3: usbc-gnd -> led10-vcc
- U26 pad 4: led9.ic-vcc -> led9-vcc
Routing:
- net (no net): track 2391.0 -> 0.84 mm, vias 174 -> 0
- net vcc: track 0.00 -> 22.8 mm, vias 0 -> 3
- net power_stage-vcc-3: track 0.00 -> 21.7 mm, vias 0 -> 1
- net power_stage-vcc-1: track 0.00 -> 20.8 mm, vias 0 -> 2
- net power_stage-vcc-2: track 0.00 -> 20.0 mm, vias 0 -> 2
- net power_stage-vcc-5: track 0.00 -> 19.4 mm, vias 0 -> 2
- net power_stage-vcc-4: track 0.00 -> 15.6 mm, vias 0 -> 2
- net usbc-vcc: track 33.1 -> 21.1 mm, vias 10 -> 0
- net en: track 8.40 -> 15.3 mm
- net shifter.ic-gnd: track 0.00 -> 4.91 mm
- net power_stage-vcc-6: track 0.00 -> 4.75 mm, vias 0 -> 2
- net gnd: track 0.00 -> 4.08 mm, vias 0 -> 3
- net power_stage.ic-vcc-3: track 0.00 -> 3.95 mm
- net hba.nfet_low-source: track 0.00 -> 3.37 mm
- net power_stage-vcc-7: track 0.00 -> 3.37 mm
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- added copper zone on B.Cu, net gnd
- removed copper zone on B.Cu, net (none)
- removed copper zone on F.Cu, net (none)
Other:
- outline, holes or cut-outs redrawn
- board text removed: "IN"
- board text removed: "OUT"
- board text removed: "U2"

Commit message: chugging thru layout
Parts:
- R10, R11, R8, R9: moved to B.Cu
- moved U16 76.8 mm to (114.7, 69.8), turned to 0 degrees
- moved C19 74.7 mm to (114.6, 72.7), turned to 0 degrees
- moved C2 21.1 mm to (22.1, 48.8), turned to -90 degrees
- moved C5 19.1 mm to (30.4, 98.0), turned to 180 degrees
- moved U4 16.8 mm to (35.4, 97.5), turned to 0 degrees
- moved C4 16.4 mm to (30.4, 95.9), turned to 180 degrees
- moved U2 16.0 mm to (26.6, 49.0), turned to -90 degrees
- moved C3 14.5 mm to (30.5, 94.4), turned to 180 degrees
- moved R3 13.9 mm to (33.2, 95.0), turned to 0 degrees
- moved C1 12.4 mm to (31.1, 49.0), turned to 90 degrees
- moved C12 7.58 mm to (32.0, 37.2), turned to -90 degrees
- moved R15 6.14 mm to (37.6, 25.8), turned to 180 degrees
- moved R16 6.00 mm to (25.0, 26.0)
- moved C14 5.44 mm to (40.2, 34.2), turned to 90 degrees
- moved U3 5.13 mm to (38.8, 84.0), turned to 90 degrees
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Connections:
- C10 pad 1: power_stage.ic-vcc-2 -> power_stage.ic-vcc-1
- C11 pad 1: power_stage.ic-vcc-3 -> power_stage.ic-vcc-2
- C19 pad 1: shifter.ic-vcc -> usbc-vcc
- C19 pad 2: shifter.ic-gnd -> usbc-gnd
- C8 pad 1: power_stage.bypass_cap-vcc -> usbc-vcc
- C8 pad 2: power_stage.bypass_cap-gnd -> usbc-gnd
- C9 pad 1: power_stage.ic-vcc-1 -> power_stage.ic-vcc
- Q1 pad 2: strain_adc.ic-vcc -> ldo3V3-vcc
- Q1 pad 3: ldo3V3-vcc -> strain_adc.ic-vcc
- R4 pad 1: esp32s3.ic-vcc-2 -> esp32s3.ic-vcc-4
- U14 pad 15: rate -> ldo3V3-vcc
- U16 pad 3: shifter.ic-gnd -> usbc-gnd
- U16 pad 5: shifter.ic-vcc -> usbc-vcc
- U3 pad 10: esp32s3.ic-vcc-2 -> esp32s3.ic-vcc-4
- U3 pad 11: esp32s3.ic-vcc-1 -> esp32s3.ic-vcc-3
- U3 pad 16: io46 -> esp32s3.ic-vcc-2
- U3 pad 26: io45 -> esp32s3.ic-vcc-1
- U3 pad 9: esp32s3.ic-vcc-3 -> esp32s3.ic-vcc-5
- U7 pad 1: esp32s3.ic-sda -> esp32s3.ic-vcc-1
- U7 pad 14: power_stage.ic-vcc-3 -> power_stage.ic-vcc-2
- U7 pad 17: power_stage.ic-vcc-2 -> power_stage.ic-vcc-1
- U7 pad 2: esp32s3.ic-vcc-2 -> esp32s3.ic-vcc-4
- U7 pad 20: power_stage.ic-vcc-1 -> power_stage.ic-vcc
- U7 pad 22: esp32s3.ic-vcc-3 -> esp32s3.ic-vcc-2
- U7 pad 23: esp32s3.ic-vcc-1 -> esp32s3.ic-vcc-3
- U7 pad 24: esp32s3.ic-vcc-3 -> esp32s3.ic-vcc-5
- U7 pad 25: power_stage.ic-gnd -> usbc-gnd
- U7 pad 4: power_stage.ic-vcc -> usbc-vcc
- U7 pad 6: power_stage.ic-gnd -> usbc-gnd
Routing:
- net usbc-vcc: track 21.1 -> 155.0 mm
- net esp32s3.ic-sda: track 1.77 -> 87.8 mm, vias 1 -> 0
- net p: track 0.00 -> 67.7 mm, vias 0 -> 1
- net n: track 0.00 -> 43.6 mm, vias 0 -> 1
- net scl: track 2.74 -> 38.7 mm
- net power_stage-vcc-6: track 4.75 -> 25.0 mm
- net en: track 15.3 -> 8.40 mm
- net shifter.ic-gnd: track 4.91 -> 0.00 mm
- net power_stage.ic-vcc-3: track 3.95 -> 0.00 mm
- net vcc-1: track 5.16 -> 1.44 mm
- net inna: track 0.00 -> 3.12 mm
- net inpa: track 0.00 -> 3.09 mm
- net innb: track 0.00 -> 3.06 mm
- net io11: track 2.86 -> 0.00 mm
- net io5: track 2.85 -> 0.00 mm
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- added copper zone on B.Cu, net (none)
- removed copper zone on B.Cu, net gnd
